Commit message: Expose argument to select UR and TORSO hardware interface for simulation

File: vulcano_description/robots/vulcano.urdf.xacro (robot description, xacro)
@@ -1,5 +1,5 @@
 <?xml version="1.0"?>
 <robot name="vulcano" xmlns:xacro="http://www.ros.org/wiki/xacro">
-  <xacro:macro name="vulcano" params="ur_hw_interface:=hardware_interface/PositionJointInterface">
+  <xacro:macro name="vulcano" params="hw_interface:=hardware_interface/PositionJointInterface">
     <xacro:property name="PI" value="3.1415926535897931"/>
     <xacro:arg name="joint_limited" default="false"/>
@@ -30,5 +30,5 @@
       <axis xyz="0 0 0"/>
     </joint>
-    <xacro:vulcano_torso prefix="" hq="${hq}" />
+    <xacro:vulcano_torso prefix="" hq="${hq}" transmission_hw_interface="${hw_interface}"/>
     <!-- Fix right arm to torso -->
     <joint name="torso_right_arm_base_joint" type="fixed">
@@ -38,5 +38,5 @@
     </joint>
     <!--xacro:ur10_robot prefix="right_arm_" joint_limited="$(arg joint_limited)"/-->
-    <xacro:right_arm_ur10_robot prefix="right_arm_" joint_limited="$(arg joint_limited)" transmission_hw_interface="${ur_hw_interface}"/>
+    <xacro:right_arm_ur10_robot prefix="right_arm_" joint_limited="$(arg joint_limited)" transmission_hw_interface="${hw_interface}"/>
     <!-- Fix left arm to torso -->
     <joint name="torso_left_arm_base_joint" type="fixed">
@@ -46,5 +46,5 @@
     </joint>
     <!--xacro:ur10_robot prefix="left_arm_" joint_limited="$(arg joint_limited)"/-->
-    <xacro:left_arm_ur10_robot prefix="left_arm_" joint_limited="$(arg joint_limited)" transmission_hw_interface="${ur_hw_interface}"/>
+    <xacro:left_arm_ur10_robot prefix="left_arm_" joint_limited="$(arg joint_limited)" transmission_hw_interface="${hw_interface}"/>
     <xacro:tube_support prefix="left_arm_ee_" parent="left_arm_ee_link">
       <origin xyz="0.012 0 0.0975" rpy="0 0 0"/>

File: vulcano_description/robots/vulcano_robot.urdf.xacro (robot description, xacro)
@@ -1,6 +1,6 @@
 <?xml version="1.0"?>
 <robot name="vulcano" xmlns:xacro="http://www.ros.org/wiki/xacro">
-  <xacro:arg name="ur_hw_interface" default="hardware_interface/PositionJointInterface"/>
+  <xacro:arg name="hw_interface" default="hardware_interface/PositionJointInterface"/>
   <xacro:include filename="$(find vulcano_description)/robots/vulcano.urdf.xacro"/>
-  <xacro:vulcano ur_hw_interface="$(arg ur_hw_interface)"/>
+  <xacro:vulcano hw_interface="$(arg hw_interface)"/>
 </robot>

File: vulcano_torso_description/urdf/guidance/guidance.urdf.xacro (robot description, xacro)
@@ -6,5 +6,5 @@
   <xacro:property name="z_elevation_joint" value="0.442"/>
   <!-- Define the torso -->
-  <xacro:macro name="guidance" params="prefix parent hq">
+  <xacro:macro name="guidance" params="prefix parent hq transmission_hw_interface">
     <joint name="${prefix}torso_guidance_base_joint" type="fixed">
       <origin xyz="0.0 0.0 0.0" rpy="0 0 0"/>
@@ -46,5 +46,5 @@
       <type>transmission_interface/SimpleTransmission</type>
       <joint name="${prefix}torso_guidance_revolution_joint">
-        <hardwareInterface>PositionJointInterface</hardwareInterface>
+        <hardwareInterface>${transmission_hw_interface}</hardwareInterface>
       </joint>
       <actuator name="${prefix}torso_guidance_revolution_motor">
@@ -85,5 +85,5 @@
       <type>transmission_interface/SimpleTransmission</type>
       <joint name="${prefix}torso_guidance_elevation_joint">
-        <hardwareInterface>PositionJointInterface</hardwareInterface>
+        <hardwareInterface>${transmission_hw_interface}</hardwareInterface>
       </joint>
       <actuator name="${prefix}torso_guidance_elevation_motor">

File: vulcano_torso_description/urdf/vulcano_torso.urdf.xacro (robot description, xacro)
@@ -11,5 +11,5 @@
     <xacro:include filename="$(find vulcano_torso_description)/urdf/tube_support/tube_support.urdf.xacro"/>
     <xacro:include filename="$(find robotnik_sensors)/urdf/all_sensors.urdf.xacro" />
-    <xacro:macro name="vulcano_torso" params="prefix hq"> <!-- TODO: check hq variable -->
+    <xacro:macro name="vulcano_torso" params="prefix hq transmission_hw_interface"> <!-- TODO: check hq variable -->
         <link name="${prefix}torso_base_link">
             <inertial>
@@ -19,5 +19,5 @@
             </inertial>
         </link>
-        <xacro:guidance prefix="${prefix}" parent="${prefix}torso_base_link" hq="${hq}"/>
+        <xacro:guidance prefix="${prefix}" parent="${prefix}torso_base_link" hq="${hq}" transmission_hw_interface="${hw_interface}"/>
         <joint name="${prefix}torso_guidance_pantilt_joint" type="fixed">
           <origin xyz="-0.191 0.0 1.178" rpy="0 0 ${180*deg2rad}"/>
