Commit message: Created simple collision model for Vulcano to be used in rkcl

File: vulcano_base_description/urdf/bases/base.urdf.xacro (robot description, xacro)
@@ -79,8 +79,9 @@
     </visual>
     <collision>
-       <origin xyz="0 0 0" rpy="0 0 0 " />
-       <geometry>
-         <mesh filename="package://vulcano_base_description/meshes/bases/vulcano_base_cabinet.dae"/>
-       </geometry>
+      <origin rpy="0 0 0" xyz="-0.009 -0.00005 0.32"/>
+      <geometry>
+          <!-- <mesh filename="package://vulcano_base_description/meshes/bases/vulcano_base_cabinet.dae"/> -->
+          <box size="1.3132 0.7999 0.64" />
+      </geometry>
     </collision>
   </link>

File: vulcano_calibrated_ur_description/urdf/calibrated_ur10_vulcano_left_arm.urdf.xacro (robot description, xacro)
@@ -108,6 +108,8 @@
             </visual>
             <collision>
-                <geometry>
-                    <mesh filename="package://ur_description/meshes/ur10/collision/base.stl" />
+                <origin rpy="0 0 0" xyz="0.0 -0.00845 0.019"/>
+                <geometry>
+                    <!-- <mesh filename="package://ur_description/meshes/ur10/collision/base.stl" /> -->
+                    <box size="0.15 0.1671 0.0380" />
                 </geometry>
             </collision>
@@ -162,7 +164,9 @@
             </visual>
             <collision>
-                <geometry>
-                    <mesh filename="package://ur_description/meshes/ur10/collision/shoulder.stl" />
-                </geometry>
+              <origin rpy="0 0 0" xyz="0.0 0.0053 -0.00045"/>
+              <geometry>
+                  <!-- <mesh filename="package://ur_description/meshes/ur10/collision/shoulder.stl" /> -->
+                  <box size="0.151 0.1614 0.17" />
+              </geometry>
             </collision>
             <xacro:cylinder_inertial radius="0.075" length="0.178" mass="${shoulder_mass}">
@@ -216,7 +220,9 @@
             </visual>
             <collision>
-                <geometry>
-                    <mesh filename="package://ur_description/meshes/ur10/collision/upperarm.stl" />
-                </geometry>
+              <origin rpy="0 0 0" xyz="-0.0001 -0.0464 0.29995"/>
+              <geometry>
+                  <!-- <mesh filename="package://ur_description/meshes/ur10/collision/upperarm.stl" /> -->
+                  <box size="0.1506 0.1772 0.7489" />
+              </geometry>
             </collision>
             <xacro:cylinder_inertial radius="0.075" length="${-ur10_a2}" mass="${upper_arm_mass}">
@@ -270,7 +276,9 @@
             </visual>
             <collision>
-                <geometry>
-                    <mesh filename="package://ur_description/meshes/ur10/collision/forearm.stl" />
-                </geometry>
+              <origin rpy="0 0 0" xyz="-0.0001 -0.00085 0.2804"/>
+              <geometry>
+                  <!-- <mesh filename="package://ur_description/meshes/ur10/collision/forearm.stl" /> -->
+                  <box size="0.1202 0.1363 0.6782" />
+              </geometry>
             </collision>
             <xacro:cylinder_inertial radius="0.075" length="${-ur10_a3}" mass="${forearm_mass}">
@@ -324,7 +332,9 @@
             </visual>
             <collision>
-                <geometry>
-                    <mesh filename="package://ur_description/meshes/ur10/collision/wrist1.stl" />
-                </geometry>
+              <origin rpy="0 0 0" xyz="-0.0002 0.11095 0.0026"/>
+              <geometry>
+                  <!-- <mesh filename="package://ur_description/meshes/ur10/collision/wrist1.stl" /> -->
+                  <box size="0.091 0.1001 0.1188" />
+              </geometry>
             </collision>
             <xacro:cylinder_inertial radius="0.075" length="0.12" mass="${wrist_1_mass}">
@@ -378,7 +388,9 @@
             </visual>
             <collision>
-                <geometry>
-                    <mesh filename="package://ur_description/meshes/ur10/collision/wrist2.stl" />
-                </geometry>
+              <origin rpy="0 0 0" xyz="0.00005 0.00215 0.11205"/>
+              <geometry>
+                  <!-- <mesh filename="package://ur_description/meshes/ur10/collision/wrist2.stl" /> -->
+                  <box size="0.0913 0.1189 0.1001" />
+              </geometry>
             </collision>
             <xacro:cylinder_inertial radius="0.075" length="0.12" mass="${wrist_2_mass}">
@@ -432,7 +444,9 @@
             </visual>
             <collision>
-                <geometry>
-                    <mesh filename="package://ur_description/meshes/ur10/collision/wrist3.stl" />
-                </geometry>
+              <origin rpy="0 0 0" xyz="0.0 0.07685 0.00095"/>
+              <geometry>
+                  <!-- <mesh filename="package://ur_description/meshes/ur10/collision/wrist3.stl" /> -->
+                  <box size="0.09 0.0305 0.0901" />
+              </geometry>
             </collision>
             <xacro:cylinder_inertial radius="0.075" length="0.12" mass="${wrist_3_mass}">

File: vulcano_calibrated_ur_description/urdf/calibrated_ur10_vulcano_right_arm.urdf.xacro (robot description, xacro)
@@ -108,7 +108,9 @@
             </visual>
             <collision>
-                <geometry>
-                    <mesh filename="package://ur_description/meshes/ur10/collision/base.stl" />
-                </geometry>
+              <origin rpy="0 0 0" xyz="0.0 -0.00845 0.019"/>
+              <geometry>
+                  <!-- <mesh filename="package://ur_description/meshes/ur10/collision/base.stl" /> -->
+                  <box size="0.15 0.1671 0.0380" />
+              </geometry>
             </collision>
             <xacro:cylinder_inertial radius="0.075" length="0.038" mass="${base_mass}">
@@ -162,7 +164,9 @@
             </visual>
             <collision>
-                <geometry>
-                    <mesh filename="package://ur_description/meshes/ur10/collision/shoulder.stl" />
-                </geometry>
+              <origin rpy="0 0 0" xyz="0.0 0.0053 -0.00045"/>
+              <geometry>
+                  <!-- <mesh filename="package://ur_description/meshes/ur10/collision/shoulder.stl" /> -->
+                  <box size="0.151 0.1614 0.17" />
+              </geometry>
             </collision>
             <xacro:cylinder_inertial radius="0.075" length="0.178" mass="${shoulder_mass}">
@@ -216,7 +220,9 @@
             </visual>
             <collision>
-                <geometry>
-                    <mesh filename="package://ur_description/meshes/ur10/collision/upperarm.stl" />
-                </geometry>
+              <origin rpy="0 0 0" xyz="-0.0001 -0.0464 0.29995"/>
+              <geometry>
+                  <!-- <mesh filename="package://ur_description/meshes/ur10/collision/upperarm.stl" /> -->
+                  <box size="0.1506 0.1772 0.7489" />
+              </geometry>
             </collision>
             <xacro:cylinder_inertial radius="0.075" length="${-ur10_a2}" mass="${upper_arm_mass}">
@@ -270,7 +276,9 @@
             </visual>
             <collision>
-                <geometry>
-                    <mesh filename="package://ur_description/meshes/ur10/collision/forearm.stl" />
-                </geometry>
+              <origin rpy="0 0 0" xyz="-0.0001 -0.00085 0.2804"/>
+              <geometry>
+                  <!-- <mesh filename="package://ur_description/meshes/ur10/collision/forearm.stl" /> -->
+                  <box size="0.1202 0.1363 0.6782" />
+              </geometry>
             </collision>
             <xacro:cylinder_inertial radius="0.075" length="${-ur10_a3}" mass="${forearm_mass}">
@@ -324,7 +332,9 @@
             </visual>
             <collision>
-                <geometry>
-                    <mesh filename="package://ur_description/meshes/ur10/collision/wrist1.stl" />
-                </geometry>
+              <origin rpy="0 0 0" xyz="-0.0002 0.11095 0.0026"/>
+              <geometry>
+                  <!-- <mesh filename="package://ur_description/meshes/ur10/collision/wrist1.stl" /> -->
+                  <box size="0.091 0.1001 0.1188" />
+              </geometry>
             </collision>
             <xacro:cylinder_inertial radius="0.075" length="0.12" mass="${wrist_1_mass}">
@@ -378,7 +388,9 @@
             </visual>
             <collision>
-                <geometry>
-                    <mesh filename="package://ur_description/meshes/ur10/collision/wrist2.stl" />
-                </geometry>
+              <origin rpy="0 0 0" xyz="0.00005 0.00215 0.11205"/>
+              <geometry>
+                  <!-- <mesh filename="package://ur_description/meshes/ur10/collision/wrist2.stl" /> -->
+                  <box size="0.0913 0.1189 0.1001" />
+              </geometry>
             </collision>
             <xacro:cylinder_inertial radius="0.075" length="0.12" mass="${wrist_2_mass}">
@@ -432,7 +444,9 @@
             </visual>
             <collision>
-                <geometry>
-                    <mesh filename="package://ur_description/meshes/ur10/collision/wrist3.stl" />
-                </geometry>
+              <origin rpy="0 0 0" xyz="0.0 0.07685 0.00095"/>
+              <geometry>
+                  <!-- <mesh filename="package://ur_description/meshes/ur10/collision/wrist3.stl" /> -->
+                  <box size="0.09 0.0305 0.0901" />
+              </geometry>
             </collision>
             <xacro:cylinder_inertial radius="0.075" length="0.12" mass="${wrist_3_mass}">

File: vulcano_description/robots/vulcano.urdf.xacro (robot description, xacro)
@@ -1,5 +1,5 @@
 <?xml version="1.0"?>
 <robot name="vulcano" xmlns:xacro="http://www.ros.org/wiki/xacro">
-  <xacro:macro name="vulcano" params="joint_limited:=false custom_limits:=false ur_hw_interface:=hardware_interface/PositionJointInterface">
+  <xacro:macro name="vulcano" params="joint_limited:=false custom_limits:=false hw_interface:=hardware_interface/PositionJointInterface">
     <xacro:property name="PI" value="3.1415926535897931"/>
     <xacro:arg name="joint_limited" default="false"/>

File: vulcano_torso_description/urdf/guidance/guidance.urdf.xacro (robot description, xacro)
@@ -63,7 +63,8 @@
       </visual>
       <collision>
-        <origin xyz="0 0 0" rpy="0 0 0"/>
+        <origin rpy="0 0 0" xyz="0.0 0.0 0.7165"/>
         <geometry>
-          <mesh filename="package://vulcano_torso_description/meshes/guidance/main.stl"/>
+          <!-- <mesh filename="package://vulcano_torso_description/meshes/guidance/main.stl"/> -->
+          <box size="0.286 0.286 1.4330" />
         </geometry>
       </collision>
@@ -102,7 +103,8 @@
       </visual>
       <collision>
-        <origin xyz="0 0 0" rpy="0 0 0"/>
+        <origin rpy="0 0 0" xyz="-0.19 0.0 0.29"/>
         <geometry>
-          <mesh filename="package://vulcano_torso_description/meshes/guidance/slide.stl"/>
+          <!-- <mesh filename="package://vulcano_torso_description/meshes/guidance/slide.stl"/> -->
+          <box size="0.08 0.22 0.01" />
         </geometry>
       </collision>

File: vulcano_torso_description/urdf/pantilt/pantilt.urdf.xacro (robot description, xacro)
@@ -1,3 +1,3 @@
-﻿<?xml version="1.0"?>
+<?xml version="1.0"?>
 <robot xmlns:xacro="http://ros.org/wiki/xacro">
   <xacro:property name="PI" value="3.1415926535897931"/>
@@ -218,7 +218,8 @@
       </visual>
       <collision>
-        <origin xyz="0 0 0" rpy="0 0 0"/>
-        <geometry>
-          <mesh filename="package://vulcano_torso_description/meshes/pantilt/pantilt.stl"/>
+        <origin rpy="0 0 0" xyz="0.0 0.0 -0.02225"/>
+        <geometry>
+          <!-- <mesh filename="package://vulcano_torso_description/meshes/pantilt/pantilt.stl"/> -->
+          <box size="0.1164 0.37 0.1765" />
         </geometry>
       </collision>
